File: PCB_v1/_autosave-tuner time.kicad_sch (KiCad schematic)
At the start: 0 parts

Commit message: Last push before PCB
Changed lines of the file:
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@@
 	(wire
 		(pts
-			(xy 267.97 34.29) (xy 267.97 39.37)
+			(xy 214.63 64.77) (xy 214.63 69.85)
 		)
 		(stroke
@@
 	(wire
 		(pts
-			(xy 261.62 34.29) (xy 267.97 34.29)
+			(xy 208.28 64.77) (xy 214.63 64.77)
 		)
 		(stroke
@@
 	(global_label "VBUS"
 		(shape bidirectional)
-		(at 236.22 22.86 180)
+		(at 182.88 53.34 180)
 		(fields_autoplaced yes)
 		(effects
@@
 		)
 		(property "Intersheetrefs" "${INTERSHEET_REFS}"
-			(at 227.2249 22.86 0)
+			(at 173.8849 53.34 0)
 			(effects
 				(font
@@
 	(symbol
 		(lib_id "power:GND")
-		(at 267.97 39.37 0)
+		(at 214.63 69.85 0)
 		(unit 1)
 		(exclude_from_sim no)
@@
 		(fields_autoplaced yes)
 		(property "Reference" "#PWR0107"
-			(at 267.97 45.72 0)
+			(at 214.63 76.2 0)
 			(effects
 				(font
@@
 		)
 		(property "Value" "GND"
-			(at 267.97 44.45 0)
+			(at 214.63 74.93 0)
 			(effects
 				(font
@@
 		)
 		(property "Footprint" ""
-			(at 267.97 39.37 0)
+			(at 214.63 69.85 0)
 			(effects
 				(font
@@
 		)
 		(property "Datasheet" ""
-			(at 267.97 39.37 0)
+			(at 214.63 69.85 0)
 			(effects
 				(font
@@
 		)
 		(property "Description" "Power symbol creates a global label with name \"GND\" , ground"
-			(at 267.97 39.37 0)
+			(at 214.63 69.85 0)
 			(effects
 				(font
@@
 	)
 	(sheet
-		(at 236.22 20.32)
+		(at 182.88 50.8)
 		(size 25.4 20.32)
 		(fields_autoplaced yes)
@@
 		)
 		(property "Sheetname" "USB"
-			(at 236.22 19.6084 0)
+			(at 182.88 50.0884 0)
 			(effects
 				(font
@@
 		)
 		(property "Sheetfile" "USB.kicad_sch"
-			(at 236.22 41.2246 0)
+			(at 182.88 71.7046 0)
 			(effects
 				(font
@@
 		)
 		(pin "VBUS" bidirectional
-			(at 236.22 22.86 180)
+			(at 182.88 53.34 180)
 			(effects
 				(font
@@
 		)
 		(pin "D-" bidirectional
-			(at 236.22 34.29 180)
+			(at 182.88 64.77 180)
 			(effects
 				(font
@@
 		)
 		(pin "D+" bidirectional
-			(at 236.22 31.75 180)
+			(at 182.88 62.23 180)
 			(effects
 				(font
@@
 		)
 		(pin "GND" input
-			(at 261.62 34.29 0)
-			(effects
-				(font
+			(at 208.28 64.77 0)
+			(effects
+				(font
