File: PCB_v1/tuner time.kicad_pcb (KiCad board)
At the start: 2 copper layers, 121 parts, among them J3 Conn_01x05_Pin, J4 Conn_01x05_Pin, J5 OLED Module Mount, SW7 SW_Push, SW8 SW_Push, U2 BQ27441-G1

Commit message: pcb updated
Parts:
- added IC1: MIC_I2S_SPH0645, Parts_Library:SPH0645LM4H, F.Cu at (153.5, 133.3)
- added IC2: MIC_I2S_SPH0645, Parts_Library:SPH0645LM4H, F.Cu at (153.5, 97.0)
- added IC3: FT2332RL, Parts_Library:SSOP28-LD, F.Cu at (102.2, 130.2)
- added J1: 1051640001, Parts_Library:CON00906_5_MOL, F.Cu at (98.0, 113.0)
- added J2: S2B-PH-K-SLFSN, Parts_Library:CONN_S2B-PH-K-S_JST, F.Cu at (103.0, 98.1)
- added REF**: CONN_B4B-XH-A_JST, Parts_Library:CONN_B4B-XH-A_JST, F.Cu at (151.0, 119.5)
- added U1: BQ25185DLHR, Parts_Library:WSON10_DLH_TEX, F.Cu at (107.6, 100.4)
- added U3: DRV8834PWP, Parts_Library:SOP65P640X120-25N, F.Cu at (141.5, 115.0)
- added U4: STM32F407VGT6, Parts_Library:LQFP100_14x14_STM, F.Cu at (123.1, 124.0)
- moved U2 143.6 mm to (113.6, 100.5)
- moved C14 63.6 mm to (213.3, 80.4)
- moved C15 63.6 mm to (213.3, 83.4)
- moved C16 63.6 mm to (213.3, 86.5)
- moved C17 63.6 mm to (213.3, 89.5)
- moved C18 63.6 mm to (213.3, 92.5)
- moved C19 63.6 mm to (213.3, 95.5)
- moved C20 63.6 mm to (175.9, 123.5)
- moved C21 63.6 mm to (175.9, 126.5)
- moved C23 63.6 mm to (175.9, 129.5)
- moved C24 63.6 mm to (175.9, 132.5)
- moved C25 63.6 mm to (175.9, 135.5)
- moved C26 63.6 mm to (175.9, 138.5)
- moved C41 63.6 mm to (197.4, 80.4)
- moved C42 63.6 mm to (197.4, 83.4)
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Other:
- board outline added: 60 x 40.5 mm
- copper layers 2 -> 4

Commit message: changed the MICs to JST headers
Other:
- outline, holes or cut-outs redrawn
Changed lines of the file:
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@@
 		(fp_arc
 			(start 0.22 1.33)
-			(mid -0.005 1.3708)
+			(mid -0.005001 1.3708)
 			(end -0.230001 1.33)
 			(stroke
@@
 		(fp_arc
 			(start 0.22 1.33)
-			(mid -0.005 1.3708)
+			(mid -0.005001 1.3708)
 			(end -0.230001 1.33)
 			(stroke
@@
 	)
 	(gr_rect
+		(start 135.5 129.5)
+		(end 138.5 134)
+		(stroke
+			(width 0.05)
+			(type default)
+		)
+		(fill none)
+		(layer "Edge.Cuts")
+	)
+	(gr_rect
