File: PCB_v1/tuner time.kicad_pcb (KiCad board)
At the start: 4 copper layers, 80 x 40 mm, 111 parts, among them J1 B6B-PH-K-S, J10 Conn_01x03, J11 1051640001, J2 B6B-PH-K-S, J3 JST_B2B-PH-K-S, J4 Conn_01x05_Pin, J5 Conn_01x05_Pin, J6 OLED Conn_02x04, J7 B4B-XH-A, J8 Conn_01x02_Pin, J9 Conn_02x05_Odd_Even, SW1 SW_SPST, SW2 SW_Push, SW3 SW_Push, SW4 SW_Push, SW5 SW_Push, SW6 SW_Push, SW7 SW_Push, SW8 SW_Push, SW9 SW_SPDT, U1 BQ25185DLHR, U2 BQ27441-G1, U3 SMS05T1G, U4 SMS05T1G, U5 DRV8834PWP, U6 MAX7375AXR805, U7 STM32F405RGTx, U8 ESD9B5.0ST5G

Commit message: PCB all Done no Dr.Walter Review
Parts:
- removed C13: 0.1uF, Library:C_0805_2012Metric
- removed C14: 10uF, Library:C_0805_2012Metric
- removed R21: 10k, Library:R_0805_2012Metric
- removed TP7: ~, Library:TestPoint_THTPad_D0.8mm_Drill0.4mm
- added G***: LOGO, LOGO, F.Cu at (219.4, 111.3)
- added G***: LOGO, LOGO, B.Cu at (191.6, 127.5)
- C9: value 4.7uF -> 2.2uF
- R15, R16: value 47k -> 51k
- R20: value 1 -> 10k
- moved R20 30.7 mm to (205.7, 127.5), turned to 180 degrees
- moved TP13 0.87 mm to (175.3, 126.0)
- moved RV1 0.53 mm to (172.2, 127.2)
- moved JP7 0.28 mm to (163.6, 126.8)
- moved C9 0.20 mm to (173.2, 130.9)
Connections:
- R20 pad 1: VMOT -> BOOT0
- R20 pad 2: Net-(C14-Pad1) -> GND
- SW9 pad 1: GND -> unconnected-(SW9-A-Pad1)
- SW9 pad 2: Net-(SW9-B) -> BOOT0
Routing:
- net BOOT0: track 2.73 -> 23.3 mm, vias 0 -> 2
- net Net-(SW9-B): track 18.8 -> 0.00 mm, vias 2 -> 0
- net GND: track 43.2 -> 38.6 mm, vias 33 -> 49
- net PH1-OSCOUT: track 2.04 -> 0.00 mm
- net Net-(C14-Pad1): track 1.59 -> 0.00 mm
- net AGND: track 6.00 -> 4.73 mm, vias 45 -> 52
- net /Motor/Vconfig: track 8.20 -> 9.43 mm
- net VINT: track 26.9 -> 27.9 mm
- net 3V3: track 52.2 -> 52.9 mm
- net Button5: track 29.2 -> 28.6 mm
- net VSYS: vias 5 -> 23
- net Net-(SW1-A): vias 0 -> 8
- added copper zone on In2.Cu, net AGND
- added copper zone on In2.Cu, net GND
- added copper zone on B.Cu, net Net-(SW1-A)
- added copper zone on In2.Cu, net Net-(SW1-A)
- added copper zone on B.Cu, net VSYS
Other:
- board text added: "+"
- board text added: "+ -"
- board text added: "-"
- board text added: "3.3v"
- board text added: "5V"
- board text added: "AGND"
- board text added: "B1"
- board text added: "B6"
- board text added: "ECE477 - Team11 Automatic Guitar Tunar v1.0"
- board text added: "M0"
- board text added: "M1"
- board text added: "MCU_RX"
- board text added: "MCU_TX"
- board text added: "PB4"
- board text added: "PC10"
- board text added: "PC11"
- board text added: "PC12"
- board text added: "RST"
- board text added: "S1 S2 Flt 5v 3.3v"
- board text added: "VBUS"
- board text added: "VSYS"
- board text added: "{ "ViaStitching": "0.2", "stitch_zone_0": { "HSpacing": "1", "VSpacing": "1", "HOffset": "0", "VOffset": "0", "Clearance": "0", "Randomize": false } }"

Commit message: last PCB
Parts:
- added D10: Blue, LED_SMD:LED_0805_2012Metric_Pad1.15x1.40mm_HandSolder, F.Cu at (167.9, 120.0)
- added G***: LOGO, LOGO, F.Cu at (216.2, 126.1)
- added R21: 1k, Library:R_0805_2012Metric, F.Cu at (167.9, 116.3)
- moved G*** 34.9 mm to (189.4, 129.2), turned to 90 degrees
Routing:
- net VSYS: track 10.3 -> 16.5 mm, vias 23 -> 25
- net 3V3: track 52.9 -> 55.8 mm
- net Net-(D10-K): track 0.00 -> 1.81 mm
- net BAT_EMPTY: track 53.0 -> 54.8 mm
- net Net-(U2-BIN): track 10.2 -> 11.8 mm
- net Net-(U1-TS/MR): track 13.8 -> 12.2 mm
- net VBUS: vias 0 -> 4
- net Net-(J11-VBUS): vias 0 -> 6
- net GND: vias 49 -> 50
- net AGND: vias 52 -> 54
- net 5V: vias 4 -> 8
- added copper zone on In2.Cu, net Net-(J11-VBUS)
- added copper zone on In2.Cu, net VBUS
Other:
- board text added: "3.3v bypass"
- board text added: "B2"
- board text added: "B3"
- board text added: "LR WS Data GND 3.3"
- board text added: "MOSI GND MISO 3.3v SCK DC RST CS"
- board text added: "RX"
- board text added: "S1 S2 Flt 5v 3.3v VSYS"
- board text added: "SWCLK"
- board text added: "SWDIO"
- board text added: "TX"
- board text removed: "MCU_RX"
- board text removed: "MCU_TX"
- board text removed: "S1 S2 Flt 5v 3.3v"
- board text removed: "{ "ViaStitching": "0.2", "stitch_zone_0": { "HSpacing": "1", "VSpacing": "1", "HOffset": "0", "VOffset": "0", "Clearance": "0", "Randomize": false } }"
