File: PCB_v1/Mic.kicad_sch (KiCad schematic)
At the start: 2 parts, among them J1 B6B-PH-K-S, J2 B6B-PH-K-S

Commit message: before oscilator
Parts:
- J1, J2: footprint GT_library:JST_B6B-PH-K-S -> B6B-PH-K-S:JST_B6B-PH-K-S
Changed lines of the file:
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@@
 			)
 		)
-		(property "Footprint" "GT_library:JST_B6B-PH-K-S"
+		(property "Footprint" "B6B-PH-K-S:JST_B6B-PH-K-S"
 			(at 177.8 72.39 0)
 			(effects
@@
 			)
 		)
-		(property "Footprint" "GT_library:JST_B6B-PH-K-S"
+		(property "Footprint" "B6B-PH-K-S:JST_B6B-PH-K-S"
 			(at 177.8 107.95 0)
 			(effects

Commit message: added the oscilator
Parts:
- J1, J2: footprint B6B-PH-K-S:JST_B6B-PH-K-S -> JST_B6B-PH-K-S
Changed lines of the file:
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@@
 	(label "WS"
 		(at 116.84 50.8 0)
+		(fields_autoplaced yes)
 		(effects
 			(font
@@
 	(label "BCLK"
 		(at 152.4 107.95 0)
+		(fields_autoplaced yes)
 		(effects
 			(font
@@
 	(label "WS"
 		(at 152.4 67.31 0)
+		(fields_autoplaced yes)
 		(effects
 			(font
@@
 	(label "DATA"
 		(at 152.4 69.85 0)
+		(fields_autoplaced yes)
 		(effects
 			(font
@@
 	(label "WS"
 		(at 152.4 102.87 0)
+		(fields_autoplaced yes)
 		(effects
 			(font
@@
 	(label "BCLK"
 		(at 116.84 45.72 0)
+		(fields_autoplaced yes)
 		(effects
 			(font
@@
 	(label "BCLK"
 		(at 152.4 72.39 0)
+		(fields_autoplaced yes)
 		(effects
 			(font
@@
 	(label "DATA"
 		(at 152.4 105.41 0)
+		(fields_autoplaced yes)
 		(effects
 			(font
@@
 	(label "DATA"
 		(at 116.84 48.26 0)
+		(fields_autoplaced yes)
 		(effects
 			(font
@@
 		(shape input)
 		(at 152.4 50.8 0)
+		(fields_autoplaced yes)
 		(effects
 			(font
@@
 		(shape input)
 		(at 152.4 48.26 0)
+		(fields_autoplaced yes)
 		(effects
 			(font
@@
 		(shape input)
 		(at 124.46 35.56 0)
+		(fields_autoplaced yes)
 		(effects
 			(font
@@
 		(shape input)
 		(at 144.78 35.56 0)
+		(fields_autoplaced yes)
 		(effects
 			(font
@@
 		(shape input)
 		(at 152.4 45.72 0)
+		(fields_autoplaced yes)
 		(effects
 			(font
@@
 			)
 		)
-		(property "Footprint" "B6B-PH-K-S:JST_B6B-PH-K-S"
+		(property "Footprint" "JST_B6B-PH-K-S"
 			(at 177.8 72.39 0)
 			(effects
@@
 			)
 		)
-		(property "Footprint" "B6B-PH-K-S:JST_B6B-PH-K-S"
+		(property "Footprint" "JST_B6B-PH-K-S"
 			(at 177.8 107.95 0)
 			(effects

Commit message: routing done no silkscreen
Changed lines of the file:
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@@
-	(wire
-		(pts
-			(xy 189.23 109.22) (xy 189.23 110.49)
-		)
-		(stroke
-			(width 0)
-			(type default)
-		)
-	)
 	(wire
 		(pts
