File: PCB_v1/power.kicad_sch (KiCad schematic)
At the start: 22 parts, among them J3 JST_B2B-XH-A, J4 Conn_01x05_Pin, J5 Conn_01x05_Pin, SW1 SW_SPST, U1 BQ25185DLHR, U2 BQ27441-G1

Commit message: adding the crystal
Parts:
- C1, C2, C3, C4, C5: symbol Device:C -> GT_LIbrary:C
- D4, D5: symbol Device:LED -> GT_LIbrary:LED
- J3: symbol 2025-02-12_12-07-11:S2B-PH-K-SLFSN -> GT_LIbrary:S2B-PH-K-SLFSN
- J4, J5: symbol Connector:Conn_01x05_Pin -> GT_LIbrary:Conn_01x05_Pin
- R10, R11, R12, R4, R5, R6, R7, R8, R9: symbol Device:R -> GT_LIbrary:R
- SW1: symbol Switch:SW_SPST -> GT_LIbrary:SW_SPST
- U1: symbol 2025-02-12_10-55-39:BQ25185DLHR -> GT_LIbrary:BQ25185DLHR
- U2: symbol Battery_Management:BQ27441-G1 -> GT_LIbrary:BQ27441-G1
Changed lines of the file:
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@@
 	)
 	(symbol
-		(lib_id "Device:R")
+		(lib_id "GT_LIbrary:R")
 		(at 26.67 48.26 180)
 		(unit 1)
@@
 	)
 	(symbol
-		(lib_id "Device:C")
+		(lib_id "GT_LIbrary:C")
 		(at 67.31 55.88 0)
 		(unit 1)
@@
 	)
 	(symbol
-		(lib_id "power:GND")
+		(lib_id "GT_LIbrary:GND")
 		(at 135.89 67.31 0)
 		(unit 1)
@@
 	)
 	(symbol
-		(lib_id "ai_breakout_ft232RL-eagle-import:5V")
+		(lib_id "GT_LIbrary:5V")
 		(at 172.72 59.69 0)
 		(unit 1)
@@
 	)
 	(symbol
-		(lib_id "power:GND")
+		(lib_id "GT_LIbrary:GND")
 		(at 60.96 146.05 0)
 		(unit 1)
@@
 	)
 	(symbol
-		(lib_id "power:GND")
+		(lib_id "GT_LIbrary:GND")
 		(at 55.88 52.07 0)
 		(unit 1)
@@
 	)
 	(symbol
-		(lib_id "Device:R")
+		(lib_id "GT_LIbrary:R")
 		(at 52.07 101.6 0)
 		(unit 1)
@@
 	)
 	(symbol
-		(lib_id "Device:C")
+		(lib_id "GT_LIbrary:C")
 		(at 116.84 101.6 0)
 		(unit 1)
@@
 	)
 	(symbol
-		(lib_id "Device:R")
+		(lib_id "GT_LIbrary:R")
 		(at 69.85 118.11 90)
 		(unit 1)
@@
 	)
 	(symbol
-		(lib_id "power:GND")
+		(lib_id "GT_LIbrary:GND")
 		(at 93.98 137.16 0)
 		(unit 1)
@@
 	)
 	(symbol
-		(lib_id "power:GND")
+		(lib_id "GT_LIbrary:GND")
 		(at 125.73 41.91 180)
 		(unit 1)
@@
 	)
 	(symbol
-		(lib_id "power:+3.3V")
+		(lib_id "GT_LIbrary:+3.3V")
 		(at 67.31 25.4 0)
 		(unit 1)
@@
 	)
 	(symbol
-		(lib_id "Battery_Management:BQ27441-G1")
+		(lib_id "GT_LIbrary:BQ27441-G1")
 		(at 95.25 115.57 0)
 		(unit 1)
@@
 	)
 	(symbol
-		(lib_id "power:GND")
+		(lib_id "GT_LIbrary:GND")
 		(at 116.84 106.68 0)
 		(unit 1)
@@
 	)
 	(symbol
-		(lib_id "power:+3.3V")
+		(lib_id "GT_LIbrary:+3.3V")
 		(at 26.67 33.02 0)
 		(unit 1)
@@
 	)
 	(symbol
-		(lib_id "ai_breakout_ft232RL-eagle-import:5V")
+		(lib_id "GT_LIbrary:5V")
 		(at 205.74 101.6 0)
 		(unit 1)
@@
 	)
 	(symbol
-		(lib_id "Device:R")
+		(lib_id "GT_LIbrary:R")
 		(at 135.89 58.42 0)
 		(unit 1)
@@
 	)
 	(symbol
-		(lib_id "power:+3.3V")
+		(lib_id "GT_LIbrary:+3.3V")
 		(at 54.61 44.45 0)
 		(unit 1)
@@
 	)
 	(symbol
-		(lib_id "Switch:SW_SPST")
+		(lib_id "GT_LIbrary:SW_SPST")
 		(at 55.88 135.89 0)
 		(unit 1)
@@
 	)
 	(symbol
-		(lib_id "power:VCC")
+		(lib_id "GT_LIbrary:VCC")
 		(at 132.08 101.6 0)
 		(unit 1)
@@
 	)
 	(symbol
-		(lib_id "power:GND")
+		(lib_id "GT_LIbrary:GND")
 		(at 123.19 30.48 0)
 		(unit 1)
@@
 	)
 	(symbol
-		(lib_id "Device:R")
+		(lib_id "GT_LIbrary:R")
 		(at 35.56 48.26 180)
 		(unit 1)
@@
 	)
 	(symbol
-		(lib_id "power:GND")
+		(lib_id "GT_LIbrary:GND")
 		(at 179.07 34.29 0)
 		(unit 1)
@@
 	)
 	(symbol
-		(lib_id "power:VCC")
+		(lib_id "GT_LIbrary:VCC")
 		(at 48.26 93.98 0)
 		(unit 1)
@@
 	)
 	(symbol
-		(lib_id "power:+3.3V")
+		(lib_id "GT_LIbrary:+3.3V")
 		(at 170.18 40.64 0)
 		(unit 1)
@@
 	)
 	(symbol
-		(lib_id "Device:R")
+		(lib_id "GT_LIbrary:R")
 		(at 125.73 58.42 0)
 		(unit 1)
@@
 	)
 	(symbol
-		(lib_id "power:+3.3V")
+		(lib_id "GT_LIbrary:+3.3V")
 		(at 35.56 33.02 0)
 		(unit 1)
@@
 	)
 	(symbol
-		(lib_id "power:GND")
+		(lib_id "GT_LIbrary:GND")
 		(at 36.83 144.78 0)
 		(unit 1)
@@
 	)
 	(symbol
-		(lib_id "Device:C")
+		(lib_id "GT_LIbrary:C")
 		(at 60.96 139.7 180)
 		(unit 1)
@@
 	)
 	(symbol
-		(lib_id "power:GND")
+		(lib_id "GT_LIbrary:GND")
 		(at 60.96 36.83 0)
 		(unit 1)
@@
 	)
 	(symbol
-		(lib_id "power:GND")
+		(lib_id "GT_LIbrary:GND")
 		(at 181.61 118.11 0)
 		(unit 1)
@@
 	)
 	(symbol
-		(lib_id "Device:C")
+		(lib_id "GT_LIbrary:C")
 		(at 60.96 33.02 0)
 		(unit 1)
@@
 	)
 	(symbol
-		(lib_id "Device:C")
+		(lib_id "GT_LIbrary:C")
 		(at 129.54 34.29 0)
 		(unit 1)
@@
 	)
 	(symbol
-		(lib_id "power:GND")
+		(lib_id "GT_LIbrary:GND")
 		(at 125.73 67.31 0)
 		(unit 1)
@@
 	)
 	(symbol
-		(lib_id "power:GND")
+		(lib_id "GT_LIbrary:GND")
 		(at 181.61 102.87 0)
 		(unit 1)
@@
 	)
 	(symbol
-		(lib_id "2025-02-12_12-07-11:S2B-PH-K-SLFSN")
+		(lib_id "GT_LIbrary:S2B-PH-K-SLFSN")
 		(at 34.29 140.97 180)
 		(unit 1)
@@
 	)
 	(symbol
-		(lib_id "power:GND")
+		(lib_id "GT_LIbrary:GND")
 		(at 172.72 69.85 0)
 		(unit 1)
@@
 	)
 	(symbol
-		(lib_id "Connector:Conn_01x05_Pin")
+		(lib_id "GT_LIbrary:Conn_01x05_Pin")
 		(at 205.74 73.66 180)
 		(unit 1)
@@
 	)
 	(symbol
-		(lib_id "power:+3.3V")
+		(lib_id "GT_LIbrary:+3.3V")
 		(at 77.47 95.25 0)
 		(unit 1)
@@
 	)
 	(symbol
-		(lib_id "Device:R")
+		(lib_id "GT_LIbrary:R")
 		(at 44.45 101.6 0)
 		(unit 1)
@@
 	)
 	(symbol
-		(lib_id "power:GND")
+		(lib_id "GT_LIbrary:GND")
 		(at 69.85 63.5 0)
 		(unit 1)
@@
 	)
 	(symbol
-		(lib_id "ai_breakout_ft232RL-eagle-import:3V3")
+		(lib_id "GT_LIbrary:3V3")
 		(at 175.26 24.13 0)
 		(unit 1)
@@
 	)
 	(symbol
-		(lib_id "Device:LED")
+		(lib_id "GT_LIbrary:LED")
 		(at 35.56 38.1 90)
 		(unit 1)
@@
 	)
 	(symbol
-		(lib_id "2025-02-12_10-55-39:BQ25185DLHR")
+		(lib_id "GT_LIbrary:BQ25185DLHR")
 		(at 72.39 41.91 0)
 		(unit 1)
@@
 	)
 	(symbol
-		(lib_id "Device:R")
+		(lib_id "GT_LIbrary:R")
 		(at 78.74 132.08 0)
 		(unit 1)
@@
 	)
 	(symbol
-		(lib_id "Connector:Conn_01x05_Pin")
+		(lib_id "GT_LIbrary:Conn_01x05_Pin")
 		(at 204.47 39.37 180)
 		(unit 1)
@@
 	)
 	(symbol
-		(lib_id "Device:R")
+		(lib_id "GT_LIbrary:R")
 		(at 132.08 109.22 0)
 		(unit 1)
@@
 	)
 	(symbol
-		(lib_id "Device:LED")
+		(lib_id "GT_LIbrary:LED")
 		(at 26.67 38.1 90)
 		(unit 1)
@@
 	)
 	(symbol
-		(lib_id "power:VCC")
+		(lib_id "GT_LIbrary:VCC")
 		(at 161.29 101.6 0)
 		(unit 1)
@@
 	)
 	(symbol
-		(lib_id "power:+3.3V")
+		(lib_id "GT_LIbrary:+3.3V")
 		(at 165.1 74.93 0)
 		(unit 1)
