File: PCB_v1/power.kicad_sch (KiCad schematic)
At the start: 22 parts, among them J3 JST_B2B-XH-A, J4 Conn_01x05_Pin, J5 Conn_01x05_Pin, SW1 SW_SPST, U1 BQ25185DLHR, U2 BQ27441-G1

Commit message: before oscilator
Parts:
- J3: footprint JST_B2B-XH-A -> CONN_S2B-PH-K-S_JST
Changed lines of the file:
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@@
 			)
 		)
-		(property "Footprint" "JST_B2B-XH-A"
+		(property "Footprint" "CONN_S2B-PH-K-S_JST"
 			(at 34.29 140.97 0)
 			(effects
@@
 			)
 		)
-		(property "Datasheet" ""
+		(property "Datasheet" "S2B-PH-K-SLFSN"
 			(at 34.29 140.97 0)
 			(effects

Commit message: added the oscilator
Parts:
- D4, D5: footprint LED_SMD:LED_0805_2012Metric_Pad1.15x1.40mm_HandSolder -> LED_0805_2012Metric_Pad1.15x1.40mm_HandSolder
- U2: footprint Package_SON:Texas_S-PDSO-N12 -> Texas_S-PDSO-N12
Changed lines of the file:
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@@
 		(shape input)
 		(at 187.96 116.84 0)
+		(fields_autoplaced yes)
 		(effects
 			(font
@@
 		(shape input)
 		(at 167.64 101.6 0)
+		(fields_autoplaced yes)
 		(effects
 			(font
@@
 		(shape bidirectional)
 		(at 39.37 110.49 180)
+		(fields_autoplaced yes)
 		(effects
 			(font
@@
 		(shape bidirectional)
 		(at 134.62 115.57 0)
+		(fields_autoplaced yes)
 		(effects
 			(font
@@
 		(shape input)
 		(at 212.09 101.6 0)
+		(fields_autoplaced yes)
 		(effects
 			(font
@@
 		(shape bidirectional)
 		(at 134.62 44.45 0)
+		(fields_autoplaced yes)
 		(effects
 			(font
@@
 		(shape input)
 		(at 187.96 101.6 0)
+		(fields_autoplaced yes)
 		(effects
 			(font
@@
 		(shape bidirectional)
 		(at 39.37 113.03 180)
+		(fields_autoplaced yes)
 		(effects
 			(font
@@
 			)
 		)
-		(property "Footprint" "Package_SON:Texas_S-PDSO-N12"
+		(property "Footprint" "Texas_S-PDSO-N12"
 			(at 101.6 129.54 0)
 			(effects
@@
 			)
 		)
-		(property "Footprint" "LED_SMD:LED_0805_2012Metric_Pad1.15x1.40mm_HandSolder"
+		(property "Footprint" "LED_0805_2012Metric_Pad1.15x1.40mm_HandSolder"
 			(at 35.56 38.1 0)
 			(effects
@@
 			)
 		)
-		(property "Footprint" "LED_SMD:LED_0805_2012Metric_Pad1.15x1.40mm_HandSolder"
+		(property "Footprint" "LED_0805_2012Metric_Pad1.15x1.40mm_HandSolder"
 			(at 26.67 38.1 0)
 			(effects

Commit message: before major move
Parts:
- J3: value JST_B2B-XH-A -> JST_B2B-PH-K-S; footprint CONN_S2B-PH-K-S_JST -> JST_B2B-PH-K-S
Changed lines of the file:
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@@
 		(dnp no)
 		(property "Reference" "R7"
-			(at 54.61 100.3299 0)
+			(at 53.594 100.33 0)
 			(effects
 				(font
@@
 		)
 		(property "Value" "5.1k"
-			(at 54.61 102.8699 0)
+			(at 53.594 102.87 0)
 			(effects
 				(font
@@
 			)
 		)
-		(property "Value" "JST_B2B-XH-A"
+		(property "Value" "JST_B2B-PH-K-S"
 			(at 25.4 133.35 0)
 			(effects
@@
 			)
 		)
-		(property "Footprint" "CONN_S2B-PH-K-S_JST"
+		(property "Footprint" "JST_B2B-PH-K-S"
 			(at 34.29 140.97 0)
 			(effects
@@
 		(on_board yes)
 		(dnp no)
-		(fields_autoplaced yes)
 		(property "Reference" "R6"
-			(at 46.99 100.3299 0)
+			(at 45.974 100.584 0)
 			(effects
 				(font
@@
 		)
 		(property "Value" "5.1k"
-			(at 46.99 102.8699 0)
-			(effects
-				(font
+			(at 45.974 102.87 0)
+			(effects
+				(font

Commit message: done no text before stiching via
Parts:
- C1, C2, C3, C4, C5: footprint Capacitor_SMD:C_0805_2012Metric -> Library:C_0805_2012Metric
- R10, R11, R12, R4, R5, R6, R7, R8, R9: footprint Resistor_SMD:R_0805_2012Metric -> Library:R_0805_2012Metric
Changed lines of the file:
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@@
 			)
 		)
-		(property "Footprint" "Resistor_SMD:R_0805_2012Metric"
+		(property "Footprint" "Library:R_0805_2012Metric"
 			(at 28.448 48.26 90)
 			(effects
@@
 			)
 		)
-		(property "Footprint" "Capacitor_SMD:C_0805_2012Metric"
+		(property "Footprint" "Library:C_0805_2012Metric"
 			(at 68.2752 59.69 0)
 			(effects
@@
 			)
 		)
-		(property "Footprint" "Resistor_SMD:R_0805_2012Metric"
+		(property "Footprint" "Library:R_0805_2012Metric"
 			(at 50.292 101.6 90)
 			(effects
@@
 			)
 		)
-		(property "Footprint" "Capacitor_SMD:C_0805_2012Metric"
+		(property "Footprint" "Library:C_0805_2012Metric"
 			(at 117.8052 105.41 0)
 			(effects
@@
 			)
 		)
-		(property "Footprint" "Resistor_SMD:R_0805_2012Metric"
+		(property "Footprint" "Library:R_0805_2012Metric"
 			(at 69.85 119.888 90)
 			(effects
@@
 			)
 		)
-		(property "Footprint" "Resistor_SMD:R_0805_2012Metric"
+		(property "Footprint" "Library:R_0805_2012Metric"
 			(at 134.112 58.42 90)
 			(effects
@@
 			)
 		)
-		(property "Footprint" "Resistor_SMD:R_0805_2012Metric"
+		(property "Footprint" "Library:R_0805_2012Metric"
 			(at 37.338 48.26 90)
 			(effects
@@
 			)
 		)
-		(property "Footprint" "Resistor_SMD:R_0805_2012Metric"
+		(property "Footprint" "Library:R_0805_2012Metric"
 			(at 123.952 58.42 90)
 			(effects
@@
 			)
 		)
-		(property "Footprint" "Capacitor_SMD:C_0805_2012Metric"
+		(property "Footprint" "Library:C_0805_2012Metric"
 			(at 59.9948 135.89 0)
 			(effects
@@
 			)
 		)
-		(property "Footprint" "Capacitor_SMD:C_0805_2012Metric"
+		(property "Footprint" "Library:C_0805_2012Metric"
 			(at 61.9252 36.83 0)
 			(effects
@@
 			)
 		)
-		(property "Footprint" "Capacitor_SMD:C_0805_2012Metric"
+		(property "Footprint" "Library:C_0805_2012Metric"
 			(at 130.5052 38.1 0)
 			(effects
@@
 			)
 		)
-		(property "Footprint" "Resistor_SMD:R_0805_2012Metric"
+		(property "Footprint" "Library:R_0805_2012Metric"
 			(at 42.672 101.6 90)
 			(effects
@@
 			)
 		)
-		(property "Footprint" "Resistor_SMD:R_0805_2012Metric"
+		(property "Footprint" "Library:R_0805_2012Metric"
 			(at 76.962 132.08 90)
 			(effects
@@
 			)
 		)
-		(property "Footprint" "Resistor_SMD:R_0805_2012Metric"
+		(property "Footprint" "Library:R_0805_2012Metric"
 			(at 130.302 109.22 90)
 			(effects

Commit message: last PCB
Parts:
- added D10: Blue, LED_0805_2012Metric_Pad1.15x1.40mm_HandSolder, symbol GT_LIbrary:LED
- added R21: 1k, Library:R_0805_2012Metric, symbol GT_LIbrary:R
Connections:
- net GND: now also R21.1
- net VSYS: now also D10.2 (A)
- new net: D10.1 (K), R21.2
