File: PCB_v1/tuner time.kicad_sch (KiCad schematic)
At the start: 15 parts

Commit message: adding the crystal
Parts:
- D1, D2, D3: symbol Device:LED -> GT_LIbrary:LED
- H1, H2: symbol Mechanical:MountingHole -> GT_LIbrary:MountingHole
- JP1: symbol Jumper:SolderJumper_2_Bridged -> GT_LIbrary:SolderJumper_2_Bridged
- JP2, JP3: symbol Jumper:SolderJumper_3_Open -> GT_LIbrary:SolderJumper_3_Open
- JP4: symbol Jumper:SolderJumper_3_Bridged12 -> GT_LIbrary:SolderJumper_3_Bridged12
- R1, R2: symbol Device:R -> GT_LIbrary:R
- R3: symbol Device:R_US -> GT_LIbrary:R_US
- TP1, TP2: symbol Connector:TestPoint -> GT_LIbrary:TestPoint
Changed lines of the file:
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@@
 	)
 	(symbol
-		(lib_id "power:GND")
+		(lib_id "GT_LIbrary:GND")
 		(at 82.55 144.78 0)
 		(unit 1)
@@
 	)
 	(symbol
-		(lib_id "power:GND")
+		(lib_id "GT_LIbrary:GND")
 		(at 149.86 62.23 0)
 		(unit 1)
@@
 	)
 	(symbol
-		(lib_id "power:VCC")
+		(lib_id "GT_LIbrary:VCC")
 		(at 154.94 30.48 0)
 		(unit 1)
@@
 	)
 	(symbol
-		(lib_id "Device:R")
+		(lib_id "GT_LIbrary:R")
 		(at 123.19 24.13 90)
 		(unit 1)
@@
 	)
 	(symbol
-		(lib_id "power:VCC")
+		(lib_id "GT_LIbrary:VCC")
 		(at 73.66 132.08 0)
 		(unit 1)
@@
 	)
 	(symbol
-		(lib_id "power:GND")
+		(lib_id "GT_LIbrary:GND")
 		(at 160.02 41.91 0)
 		(unit 1)
@@
 	)
 	(symbol
-		(lib_id "Jumper:SolderJumper_2_Bridged")
+		(lib_id "GT_LIbrary:SolderJumper_2_Bridged")
 		(at 143.51 60.96 0)
 		(unit 1)
@@
 	)
 	(symbol
-		(lib_id "power:VCC")
+		(lib_id "GT_LIbrary:VCC")
 		(at 80.01 128.27 0)
 		(unit 1)
@@
 	)
 	(symbol
-		(lib_id "Connector:TestPoint")
+		(lib_id "GT_LIbrary:TestPoint")
 		(at 232.41 76.2 270)
 		(unit 1)
@@
 	)
 	(symbol
-		(lib_id "Jumper:SolderJumper_3_Open")
+		(lib_id "GT_LIbrary:SolderJumper_3_Open")
 		(at 240.03 90.17 270)
 		(unit 1)
@@
 	)
 	(symbol
-		(lib_id "Device:LED")
+		(lib_id "GT_LIbrary:LED")
 		(at 133.35 24.13 0)
 		(unit 1)
@@
 	)
 	(symbol
-		(lib_id "Device:LED")
+		(lib_id "GT_LIbrary:LED")
 		(at 133.35 33.02 0)
 		(unit 1)
@@
 	)
 	(symbol
-		(lib_id "Device:R")
+		(lib_id "GT_LIbrary:R")
 		(at 123.19 33.02 90)
 		(unit 1)
@@
 	)
 	(symbol
-		(lib_id "power:GND")
+		(lib_id "GT_LIbrary:GND")
 		(at 224.79 111.76 0)
 		(unit 1)
@@
 	)
 	(symbol
-		(lib_id "power:VCC")
+		(lib_id "GT_LIbrary:VCC")
 		(at 176.53 76.2 0)
 		(unit 1)
@@
 	)
 	(symbol
-		(lib_id "power:GND")
+		(lib_id "GT_LIbrary:GND")
 		(at 214.63 154.94 0)
 		(unit 1)
@@
 	)
 	(symbol
-		(lib_id "Jumper:SolderJumper_3_Open")
+		(lib_id "GT_LIbrary:SolderJumper_3_Open")
 		(at 247.65 87.63 270)
 		(unit 1)
@@
 	)
 	(symbol
-		(lib_id "power:VCC")
+		(lib_id "GT_LIbrary:VCC")
 		(at 138.43 33.02 0)
 		(unit 1)
@@
 	)
 	(symbol
-		(lib_id "Mechanical:MountingHole")
+		(lib_id "GT_LIbrary:MountingHole")
 		(at 19.05 17.78 0)
 		(unit 1)
@@
 	)
 	(symbol
-		(lib_id "power:VCC")
+		(lib_id "GT_LIbrary:VCC")
 		(at 180.34 71.12 0)
 		(unit 1)
@@
 	)
 	(symbol
-		(lib_id "power:GND")
+		(lib_id "GT_LIbrary:GND")
 		(at 267.97 39.37 0)
 		(unit 1)
@@
 	)
 	(symbol
-		(lib_id "Jumper:SolderJumper_3_Bridged12")
+		(lib_id "GT_LIbrary:SolderJumper_3_Bridged12")
 		(at 254 81.28 270)
 		(unit 1)
@@
 	)
 	(symbol
-		(lib_id "power:VCC")
+		(lib_id "GT_LIbrary:VCC")
 		(at 243.84 78.74 0)
 		(unit 1)
@@
 	)
 	(symbol
-		(lib_id "power:GND")
+		(lib_id "GT_LIbrary:GND")
 		(at 116.84 39.37 0)
 		(unit 1)
@@
 	)
 	(symbol
-		(lib_id "Device:LED")
+		(lib_id "GT_LIbrary:LED")
 		(at 224.79 97.79 90)
 		(unit 1)
@@
 	)
 	(symbol
-		(lib_id "power:VCC")
+		(lib_id "GT_LIbrary:VCC")
 		(at 218.44 146.05 270)
 		(unit 1)
@@
 	)
 	(symbol
-		(lib_id "Mechanical:MountingHole")
+		(lib_id "GT_LIbrary:MountingHole")
 		(at 19.05 24.13 0)
 		(unit 1)
@@
 	)
 	(symbol
-		(lib_id "power:GND")
+		(lib_id "GT_LIbrary:GND")
 		(at 254 87.63 0)
 		(unit 1)
@@
 	)
 	(symbol
-		(lib_id "power:GND")
+		(lib_id "GT_LIbrary:GND")
 		(at 198.12 91.44 0)
 		(unit 1)
@@
 	)
 	(symbol
-		(lib_id "power:VCC")
+		(lib_id "GT_LIbrary:VCC")
 		(at 138.43 24.13 0)
 		(unit 1)
@@
 	)
 	(symbol
-		(lib_id "power:GND")
+		(lib_id "GT_LIbrary:GND")
 		(at 166.37 54.61 0)
 		(unit 1)
@@
 	)
 	(symbol
-		(lib_id "power:GND")
+		(lib_id "GT_LIbrary:GND")
 		(at 138.43 62.23 0)
 		(unit 1)
@@
 	)
 	(symbol
-		(lib_id "power:GND")
+		(lib_id "GT_LIbrary:GND")
 		(at 80.01 76.2 0)
 		(unit 1)
@@
 	)
 	(symbol
-		(lib_id "power:VCC")
+		(lib_id "GT_LIbrary:VCC")
 		(at 254 74.93 0)
 		(unit 1)
@@
 	)
 	(symbol
-		(lib_id "Connector:TestPoint")
+		(lib_id "GT_LIbrary:TestPoint")
 		(at 199.39 80.01 90)
 		(unit 1)
@@
 	)
 	(symbol
-		(lib_id "power:VCC")
+		(lib_id "GT_LIbrary:VCC")
 		(at 80.01 60.96 0)
 		(unit 1)
@@
 	)
 	(symbol
-		(lib_id "Device:R_US")
+		(lib_id "GT_LIbrary:R_US")
 		(at 224.79 106.68 0)
 		(mirror y)
@@
 	)
 	(symbol
-		(lib_id "power:GND")
+		(lib_id "GT_LIbrary:GND")
 		(at 243.84 97.79 0)
 		(unit 1)
@@
 	)
 	(symbol
-		(lib_id "power:VCC")
+		(lib_id "GT_LIbrary:VCC")
 		(at 198.12 72.39 0)
 		(unit 1)
@@
 	)
 	(symbol
-		(lib_id "power:VCC")
+		(lib_id "GT_LIbrary:VCC")
 		(at 160.02 26.67 0)
 		(unit 1)
