File: PCB_v1/oled.kicad_sch (KiCad schematic)
At the start: 17 parts, among them J6 Conn_02x04_Odd_Even, SW2 SW_Push, SW3 SW_Push, SW4 SW_Push, SW5 SW_Push, SW6 SW_Push, SW7 SW_Push, U7 SMS05T1G, U8 SMS05T1G

Commit message: pushing BOM
Parts:
- C6, C7: MFP (none) -> CA0612KRX7R7BB104
- J6: value Conn_02x04_Odd_Even -> OLED Conn_02x04; footprint Connector_PinHeader_2.00mm:PinHeader_2x04_P2.00mm_Vertical -> Connector_PinHeader_2.54mm:PinHeader_2x04_P2.54mm_Vertical; MFP (none) -> Genereic 2x4 2.56 mm
- RN2: MFP (none) -> EXB-2HV103JV
- TP3, TP4, TP5, TP6: MFP (none) -> N/A
- U3: renamed from U7; MFP (none) -> SMS05T1G
- U4: renamed from U8; MFP (none) -> SMS05T1G

Commit message: adding the crystal
Parts:
- J6: symbol Connector_Generic:Conn_02x04_Odd_Even -> GT_LIbrary:Conn_02x04_Odd_Even
- RN1, RN2: symbol Device:R_Pack08_Split -> GT_LIbrary:R_Pack08_Split
- SW2, SW3, SW4, SW5, SW6, SW7: symbol Switch:SW_Push -> GT_LIbrary:SW_Push
- TP3, TP4, TP5, TP6: symbol Connector:TestPoint -> GT_LIbrary:TestPoint
Changed lines of the file:
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@@
 	)
 	(symbol
-		(lib_id "power:GND")
+		(lib_id "GT_LIbrary:GND")
 		(at 20.32 82.55 270)
 		(unit 1)
@@
 	)
 	(symbol
-		(lib_id "Switch:SW_Push")
+		(lib_id "GT_LIbrary:SW_Push")
 		(at 72.39 116.84 0)
 		(unit 1)
@@
 	)
 	(symbol
-		(lib_id "Switch:SW_Push")
+		(lib_id "GT_LIbrary:SW_Push")
 		(at 72.39 33.02 0)
 		(unit 1)
@@
 	)
 	(symbol
-		(lib_id "Switch:SW_Push")
+		(lib_id "GT_LIbrary:SW_Push")
 		(at 72.39 59.69 0)
 		(unit 1)
@@
 	)
 	(symbol
-		(lib_id "power:GND")
+		(lib_id "GT_LIbrary:GND")
 		(at 90.17 96.52 0)
 		(unit 1)
@@
 	)
 	(symbol
-		(lib_id "Device:R_Pack08_Split")
+		(lib_id "GT_LIbrary:R_Pack08_Split")
 		(at 90.17 144.78 0)
 		(unit 4)
@@
 	)
 	(symbol
-		(lib_id "power:GND")
+		(lib_id "GT_LIbrary:GND")
 		(at 64.77 35.56 0)
 		(unit 1)
@@
 	)
 	(symbol
-		(lib_id "power:+3V0")
+		(lib_id "GT_LIbrary:+3V0")
 		(at 90.17 171.45 0)
 		(unit 1)
@@
 	)
 	(symbol
-		(lib_id "Device:R_Pack08_Split")
+		(lib_id "GT_LIbrary:R_Pack08_Split")
 		(at 90.17 175.26 0)
 		(unit 3)
@@
 	)
 	(symbol
-		(lib_id "power:GND")
+		(lib_id "GT_LIbrary:GND")
 		(at 90.17 186.69 0)
 		(unit 1)
@@
 	)
 	(symbol
-		(lib_id "power:GND")
+		(lib_id "GT_LIbrary:GND")
 		(at 90.17 156.21 0)
 		(unit 1)
@@
 	)
 	(symbol
-		(lib_id "power:+3V0")
+		(lib_id "GT_LIbrary:+3V0")
 		(at 90.17 25.4 0)
 		(unit 1)
@@
 	)
 	(symbol
-		(lib_id "power:VCC")
+		(lib_id "GT_LIbrary:VCC")
 		(at 128.27 73.66 0)
 		(unit 1)
@@
 	)
 	(symbol
-		(lib_id "power:GND")
+		(lib_id "GT_LIbrary:GND")
 		(at 90.17 124.46 0)
 		(unit 1)
@@
 	)
 	(symbol
-		(lib_id "power:+3V0")
+		(lib_id "GT_LIbrary:+3V0")
 		(at 90.17 109.22 0)
 		(unit 1)
@@
 	)
 	(symbol
-		(lib_id "Switch:SW_Push")
+		(lib_id "GT_LIbrary:SW_Push")
 		(at 72.39 148.59 0)
 		(unit 1)
@@
 	)
 	(symbol
-		(lib_id "power:+3V0")
+		(lib_id "GT_LIbrary:+3V0")
 		(at 179.07 130.81 0)
 		(unit 1)
@@
 	)
 	(symbol
-		(lib_id "Connector_Generic:Conn_02x04_Odd_Even")
+		(lib_id "GT_LIbrary:Conn_02x04_Odd_Even")
 		(at 142.24 44.45 0)
 		(unit 1)
@@
 	)
 	(symbol
-		(lib_id "Device:R_Pack08_Split")
+		(lib_id "GT_LIbrary:R_Pack08_Split")
 		(at 90.17 55.88 0)
 		(unit 7)
@@
 	)
 	(symbol
-		(lib_id "power:+3V0")
+		(lib_id "GT_LIbrary:+3V0")
 		(at 179.07 96.52 0)
 		(unit 1)
@@
 	)
 	(symbol
-		(lib_id "Connector:TestPoint")
+		(lib_id "GT_LIbrary:TestPoint")
 		(at 194.31 139.7 270)
 		(unit 1)
@@
 	)
 	(symbol
-		(lib_id "power:GND")
+		(lib_id "GT_LIbrary:GND")
 		(at 64.77 181.61 0)
 		(unit 1)
@@
 	)
 	(symbol
-		(lib_id "power:GND")
+		(lib_id "GT_LIbrary:GND")
 		(at 90.17 40.64 0)
 		(unit 1)
@@
 	)
 	(symbol
-		(lib_id "power:GND")
+		(lib_id "GT_LIbrary:GND")
 		(at 179.07 148.59 0)
 		(unit 1)
@@
 	)
 	(symbol
-		(lib_id "power:GND")
+		(lib_id "GT_LIbrary:GND")
 		(at 64.77 91.44 0)
 		(unit 1)
@@
 	)
 	(symbol
-		(lib_id "Device:R_Pack08_Split")
+		(lib_id "GT_LIbrary:R_Pack08_Split")
 		(at 90.17 85.09 0)
 		(unit 6)
@@
 	)
 	(symbol
-		(lib_id "power:GND")
+		(lib_id "GT_LIbrary:GND")
 		(at 64.77 62.23 0)
 		(unit 1)
@@
 	)
 	(symbol
-		(lib_id "power:GND")
+		(lib_id "GT_LIbrary:GND")
 		(at 64.77 119.38 0)
 		(unit 1)
@@
 	)
 	(symbol
-		(lib_id "power:GND")
+		(lib_id "GT_LIbrary:GND")
 		(at 90.17 67.31 0)
 		(unit 1)
@@
 	)
 	(symbol
-		(lib_id "Device:R_Pack08_Split")
+		(lib_id "GT_LIbrary:R_Pack08_Split")
 		(at 83.82 179.07 90)
 		(unit 6)
@@
 	)
 	(symbol
-		(lib_id "power:GND")
+		(lib_id "GT_LIbrary:GND")
 		(at 179.07 115.57 0)
 		(unit 1)
@@
 	)
 	(symbol
-		(lib_id "Device:R_Pack08_Split")
+		(lib_id "GT_LIbrary:R_Pack08_Split")
 		(at 179.07 134.62 0)
 		(unit 1)
@@
 	)
 	(symbol
-		(lib_id "Device:R_Pack08_Split")
+		(lib_id "GT_LIbrary:R_Pack08_Split")
 		(at 83.82 148.59 90)
 		(unit 5)
@@
 	)
 	(symbol
-		(lib_id "Device:R_Pack08_Split")
+		(lib_id "GT_LIbrary:R_Pack08_Split")
 		(at 83.82 59.69 90)
 		(unit 2)
@@
 	)
 	(symbol
-		(lib_id "Switch:SW_Push")
+		(lib_id "GT_LIbrary:SW_Push")
 		(at 72.39 88.9 0)
 		(unit 1)
@@
 	)
 	(symbol
-		(lib_id "Connector:TestPoint")
+		(lib_id "GT_LIbrary:TestPoint")
 		(at 161.29 139.7 90)
 		(unit 1)
@@
 	)
 	(symbol
-		(lib_id "Connector:TestPoint")
+		(lib_id "GT_LIbrary:TestPoint")
 		(at 161.29 105.41 90)
 		(unit 1)
@@
 	)
 	(symbol
-		(lib_id "Device:R_Pack08_Split")
+		(lib_id "GT_LIbrary:R_Pack08_Split")
 		(at 179.07 100.33 0)
 		(unit 2)
@@
 	)
 	(symbol
-		(lib_id "power:GND")
+		(lib_id "GT_LIbrary:GND")
 		(at 64.77 151.13 0)
 		(unit 1)
@@
 	)
 	(symbol
-		(lib_id "Connector:TestPoint")
+		(lib_id "GT_LIbrary:TestPoint")
 		(at 193.04 104.14 270)
 		(unit 1)
@@
 	)
 	(symbol
-		(lib_id "Switch:SW_Push")
+		(lib_id "GT_LIbrary:SW_Push")
 		(at 72.39 179.07 0)
 		(unit 1)
@@
 	)
 	(symbol
-		(lib_id "power:GND")
+		(lib_id "GT_LIbrary:GND")
 		(at 20.32 52.07 270)
 		(unit 1)
@@
 	)
 	(symbol
-		(lib_id "Device:R_Pack08_Split")
+		(lib_id "GT_LIbrary:R_Pack08_Split")
 		(at 83.82 116.84 90)
 		(unit 4)
@@
 	)
 	(symbol
-		(lib_id "Device:R_Pack08_Split")
+		(lib_id "GT_LIbrary:R_Pack08_Split")
 		(at 90.17 29.21 0)
 		(unit 8)
@@
 	)
 	(symbol
-		(lib_id "Device:R_Pack08_Split")
+		(lib_id "GT_LIbrary:R_Pack08_Split")
 		(at 171.45 105.41 90)
 		(unit 7)
@@
 	)
 	(symbol
-		(lib_id "power:+3V0")
+		(lib_id "GT_LIbrary:+3V0")
 		(at 90.17 81.28 0)
 		(unit 1)
@@
 	)
 	(symbol
-		(lib_id "Device:R_Pack08_Split")
+		(lib_id "GT_LIbrary:R_Pack08_Split")
 		(at 83.82 88.9 90)
 		(unit 3)
@@
 	)
 	(symbol
-		(lib_id "power:GND")
+		(lib_id "GT_LIbrary:GND")
 		(at 58.42 52.07 90)
 		(unit 1)
@@
 	)
 	(symbol
-		(lib_id "power:+3V0")
+		(lib_id "GT_LIbrary:+3V0")
 		(at 90.17 52.07 0)
 		(unit 1)
@@
 	)
 	(symbol
-		(lib_id "Device:R_Pack08_Split")
+		(lib_id "GT_LIbrary:R_Pack08_Split")
 		(at 90.17 113.03 0)
 		(unit 5)
@@
 	)
 	(symbol
-		(lib_id "power:GND")
+		(lib_id "GT_LIbrary:GND")
 		(at 58.42 82.55 90)
 		(unit 1)
@@
 	)
 	(symbol
-		(lib_id "Device:R_Pack08_Split")
+		(lib_id "GT_LIbrary:R_Pack08_Split")
 		(at 83.82 33.02 90)
 		(unit 1)
@@
 	)
 	(symbol
-		(lib_id "Device:R_Pack08_Split")
+		(lib_id "GT_LIbrary:R_Pack08_Split")
 		(at 171.45 139.7 90)
 		(unit 8)
@@
 	)
 	(symbol
-		(lib_id "power:+3V0")
+		(lib_id "GT_LIbrary:+3V0")
 		(at 90.17 140.97 0)
 		(unit 1)
@@
 	)
 	(symbol
-		(lib_id "power:GND")
+		(lib_id "GT_LIbrary:GND")
 		(at 148.59 74.93 0)
 		(unit 1)
