File: PCB_v1/USB.kicad_sch (KiCad schematic)
At the start: 3 parts, among them J10 1051640001, U7 ESD9B5.0ST5G

Commit message: push for jtag fix
Parts:
- U7: footprint ESD9B5.0ST5G:SODFL1006X40N -> Library:SODFL1006X40N
Changed lines of the file:
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@@
 		(shape bidirectional)
 		(at 165.1 80.01 180)
-		(fields_autoplaced yes)
 		(effects
 			(font
@@
 		(shape bidirectional)
 		(at 115.57 82.55 180)
-		(fields_autoplaced yes)
 		(effects
 			(font
@@
 		(shape input)
 		(at 203.2 76.2 0)
-		(fields_autoplaced yes)
 		(effects
 			(font
@@
 		(shape bidirectional)
 		(at 165.1 77.47 180)
-		(fields_autoplaced yes)
 		(effects
 			(font
@@
 			)
 		)
-		(property "Footprint" "ESD9B5.0ST5G:SODFL1006X40N"
+		(property "Footprint" "Library:SODFL1006X40N"
 			(at 153.67 93.98 0)
 			(effects

Commit message: before major move
Parts:
- renumbered J10 to J11, U7 to U8
Changed lines of the file:
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@@
 		(dnp no)
 		(fields_autoplaced yes)
-		(property "Reference" "U7"
+		(property "Reference" "U8"
 			(at 156.21 92.7099 90)
 			(effects
@@
 			(project ""
 				(path "/353cef6a-fb6e-40d9-89f8-eb54b7aa5118/0c3109f9-2cf7-4151-a3d7-47dc50d219a6"
-					(reference "U7")
+					(reference "U8")
 					(unit 1)
 				)
@@
 		(dnp no)
 		(fields_autoplaced yes)
-		(property "Reference" "J10"
+		(property "Reference" "J11"
 			(at 173.99 64.77 0)
 			(effects
@@
 			(project "tuner time"
 				(path "/353cef6a-fb6e-40d9-89f8-eb54b7aa5118/0c3109f9-2cf7-4151-a3d7-47dc50d219a6"
-					(reference "J10")
+					(reference "J11")
 					(unit 1)
 				)
@@
 		(dnp no)
 		(fields_autoplaced yes)
-		(property "Reference" "#PWR0127"
+		(property "Reference" "#PWR0124"
 			(at 160.02 62.23 0)
 			(effects
@@
 			(project "tuner time"
 				(path "/353cef6a-fb6e-40d9-89f8-eb54b7aa5118/0c3109f9-2cf7-4151-a3d7-47dc50d219a6"
-					(reference "#PWR0127")
+					(reference "#PWR0124")
 					(unit 1)
 				)
@@
 		(dnp no)
 		(fields_autoplaced yes)
-		(property "Reference" "#PWR0126"
+		(property "Reference" "#PWR0123"
 			(at 153.67 109.22 0)
 			(effects
@@
 			(project "tuner time"
 				(path "/353cef6a-fb6e-40d9-89f8-eb54b7aa5118/0c3109f9-2cf7-4151-a3d7-47dc50d219a6"
-					(reference "#PWR0126")
+					(reference "#PWR0123")
 					(unit 1)
 				)
@@
 		(dnp no)
 		(fields_autoplaced yes)
-		(property "Reference" "#PWR0128"
+		(property "Reference" "#PWR0125"
 			(at 196.85 83.82 0)
 			(effects
@@
 			(project "tuner time"
 				(path "/353cef6a-fb6e-40d9-89f8-eb54b7aa5118/0c3109f9-2cf7-4151-a3d7-47dc50d219a6"
-					(reference "#PWR0128")
+					(reference "#PWR0125")
 					(unit 1)
 				)
