File: PCB_v1/Motor.kicad_sch (KiCad schematic)
At the start: 18 parts, among them J7 B4B-XH-A, U4 DRV8834PWP

Commit message: pushing BOM
Parts:
- C10: MFP (none) -> CAP_EEE1AA101WR
- J7: MFP (none) -> B4B-XH-A
- U5: renamed from U4; MFP (none) -> DRV8834PWP
- renumbered R10 to R13, R11 to R14, R12 to R15, R13 to R16, R14 to R17, R15 to R18, R16 to R19, R17 to R20
Changed lines of the file:
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@@
 		(dnp no)
 		(fields_autoplaced yes)
-		(property "Reference" "#PWR085"
+		(property "Reference" "#PWR097"
 			(at 256.54 96.52 0)
 			(effects
@@
 			(project "tuner time"
 				(path "/353cef6a-fb6e-40d9-89f8-eb54b7aa5118/2d8cfae4-f7d1-4a7d-b5cb-7588b4c1e8a5"
-					(reference "#PWR085")
+					(reference "#PWR097")
 					(unit 1)
 				)
@@
 		(dnp no)
 		(fields_autoplaced yes)
-		(property "Reference" "R10"
+		(property "Reference" "R13"
 			(at 81.28 57.1499 0)
 			(effects
@@
 			(project "tuner time"
 				(path "/353cef6a-fb6e-40d9-89f8-eb54b7aa5118/2d8cfae4-f7d1-4a7d-b5cb-7588b4c1e8a5"
-					(reference "R10")
+					(reference "R13")
 					(unit 1)
 				)
@@
 		(dnp no)
 		(fields_autoplaced yes)
-		(property "Reference" "#PWR084"
+		(property "Reference" "#PWR096"
 			(at 245.11 93.98 0)
 			(effects
@@
 			(project "tuner time"
 				(path "/353cef6a-fb6e-40d9-89f8-eb54b7aa5118/2d8cfae4-f7d1-4a7d-b5cb-7588b4c1e8a5"
-					(reference "#PWR084")
+					(reference "#PWR096")
 					(unit 1)
 				)
@@
 		(dnp no)
 		(fields_autoplaced yes)
-		(property "Reference" "R12"
+		(property "Reference" "R15"
 			(at 143.51 119.3799 0)
 			(effects
@@
 			(project "tuner time"
 				(path "/353cef6a-fb6e-40d9-89f8-eb54b7aa5118/2d8cfae4-f7d1-4a7d-b5cb-7588b4c1e8a5"
-					(reference "R12")
+					(reference "R15")
 					(unit 1)
 				)
@@
 		(dnp no)
 		(fields_autoplaced yes)
-		(property "Reference" "R17"
+		(property "Reference" "R20"
 			(at 194.31 53.34 90)
 			(effects
@@
 			(project "tuner time"
 				(path "/353cef6a-fb6e-40d9-89f8-eb54b7aa5118/2d8cfae4-f7d1-4a7d-b5cb-7588b4c1e8a5"
-					(reference "R17")
+					(reference "R20")
 					(unit 1)
 				)
@@
 		(dnp no)
 		(fields_autoplaced yes)
-		(property "Reference" "#PWR081"
+		(property "Reference" "#PWR093"
 			(at 163.83 60.96 0)
 			(effects
@@
 			(project "tuner time"
 				(path "/353cef6a-fb6e-40d9-89f8-eb54b7aa5118/2d8cfae4-f7d1-4a7d-b5cb-7588b4c1e8a5"
-					(reference "#PWR081")
+					(reference "#PWR093")
 					(unit 1)
 				)
@@
 		(dnp no)
 		(fields_autoplaced yes)
-		(property "Reference" "#PWR078"
+		(property "Reference" "#PWR090"
 			(at 128.27 64.77 0)
 			(effects
@@
 			(project "tuner time"
 				(path "/353cef6a-fb6e-40d9-89f8-eb54b7aa5118/2d8cfae4-f7d1-4a7d-b5cb-7588b4c1e8a5"
-					(reference "#PWR078")
+					(reference "#PWR090")
 					(unit 1)
 				)
@@
 		(dnp no)
 		(fields_autoplaced yes)
-		(property "Reference" "#PWR080"
+		(property "Reference" "#PWR092"
 			(at 128.27 133.35 0)
 			(effects
@@
 			(project "tuner time"
 				(path "/353cef6a-fb6e-40d9-89f8-eb54b7aa5118/2d8cfae4-f7d1-4a7d-b5cb-7588b4c1e8a5"
-					(reference "#PWR080")
+					(reference "#PWR092")
 					(unit 1)
 				)
@@
 		(dnp no)
 		(fields_autoplaced yes)
-		(property "Reference" "#PWR076"
+		(property "Reference" "#PWR088"
 			(at 78.74 55.88 0)
 			(effects
@@
 			(project "tuner time"
 				(path "/353cef6a-fb6e-40d9-89f8-eb54b7aa5118/2d8cfae4-f7d1-4a7d-b5cb-7588b4c1e8a5"
-					(reference "#PWR076")
+					(reference "#PWR088")
 					(unit 1)
 				)
@@
 		(dnp no)
 		(fields_autoplaced yes)
-		(property "Reference" "#PWR077"
+		(property "Reference" "#PWR089"
 			(at 85.09 127 0)
 			(effects
@@
 			(project "tuner time"
 				(path "/353cef6a-fb6e-40d9-89f8-eb54b7aa5118/2d8cfae4-f7d1-4a7d-b5cb-7588b4c1e8a5"
-					(reference "#PWR077")
+					(reference "#PWR089")
 					(unit 1)
 				)
@@
 		(dnp no)
 		(fields_autoplaced yes)
-		(property "Reference" "R13"
+		(property "Reference" "R16"
 			(at 152.4 119.3799 0)
 			(effects
@@
 			(project "tuner time"
 				(path "/353cef6a-fb6e-40d9-89f8-eb54b7aa5118/2d8cfae4-f7d1-4a7d-b5cb-7588b4c1e8a5"
-					(reference "R13")
+					(reference "R16")
 					(unit 1)
 				)
@@
 		(dnp no)
 		(fields_autoplaced yes)
-		(property "Reference" "U4"
+		(property "Reference" "U5"
 			(at 105.41 58.42 0)
 			(effects
@@
 			)
 		)
-		(property "MFP" ""
+		(property "MFP" "DRV8834PWP"
 			(at 105.41 81.28 0)
 			(effects
@@
 			(project "tuner time"
 				(path "/353cef6a-fb6e-40d9-89f8-eb54b7aa5118/2d8cfae4-f7d1-4a7d-b5cb-7588b4c1e8a5"
-					(reference "U4")
+					(reference "U5")
 					(unit 1)
 				)
@@
 		(dnp no)
 		(fields_autoplaced yes)
-		(property "Reference" "#PWR083"
+		(property "Reference" "#PWR095"
 			(at 238.76 93.98 0)
 			(effects
@@
 			(project "tuner time"
 				(path "/353cef6a-fb6e-40d9-89f8-eb54b7aa5118/2d8cfae4-f7d1-4a7d-b5cb-7588b4c1e8a5"
-					(reference "#PWR083")
+					(reference "#PWR095")
 					(unit 1)
 				)
@@
 		(dnp no)
 		(fields_autoplaced yes)
-		(property "Reference" "#PWR082"
+		(property "Reference" "#PWR094"
 			(at 163.83 78.74 0)
 			(effects
@@
 			(project "tuner time"
 				(path "/353cef6a-fb6e-40d9-89f8-eb54b7aa5118/2d8cfae4-f7d1-4a7d-b5cb-7588b4c1e8a5"
-					(reference "#PWR082")
+					(reference "#PWR094")
 					(unit 1)
 				)
@@
 		(on_board yes)
 		(dnp no)
-		(property "Reference" "#PWR079"
+		(property "Reference" "#PWR091"
 			(at 128.27 120.65 0)
 			(effects
@@
 			(project "tuner time"
 				(path "/353cef6a-fb6e-40d9-89f8-eb54b7aa5118/2d8cfae4-f7d1-4a7d-b5cb-7588b4c1e8a5"
-					(reference "#PWR079")
+					(reference "#PWR091")
 					(unit 1)
 				)
@@
 		(dnp no)
 		(fields_autoplaced yes)
-		(property "Reference" "R15"
+		(property "Reference" "R18"
 			(at 162.56 116.8399 0)
 			(effects
@@
 			(project "tuner time"
 				(path "/353cef6a-fb6e-40d9-89f8-eb54b7aa5118/2d8cfae4-f7d1-4a7d-b5cb-7588b4c1e8a5"
-					(reference "R15")
+					(reference "R18")
 					(unit 1)
 				)
@@
 			)
 		)
-		(property "MFP" ""
+		(property "MFP" "B4B-XH-A"
 			(at 185.42 83.82 0)
 			(effects
@@
 		(on_board yes)
 		(dnp no)
-		(property "Reference" "R11"
+		(property "Reference" "R14"
 			(at 132.842 92.456 90)
 			(effects
@@
 			(project "tuner time"
 				(path "/353cef6a-fb6e-40d9-89f8-eb54b7aa5118/2d8cfae4-f7d1-4a7d-b5cb-7588b4c1e8a5"
-					(reference "R11")
+					(reference "R14")
 					(unit 1)
 				)
@@
 			)
 		)
-		(property "MFP" ""
+		(property "MFP" "CAP_EEE1AA101WR"
 			(at 154.94 64.77 0)
 			(effects
@@
 		(on_board yes)
 		(dnp no)
-		(property "Reference" "R14"
+		(property "Reference" "R17"
 			(at 152.4 92.71 90)
 			(effects
@@
 			(project "tuner time"
 				(path "/353cef6a-fb6e-40d9-89f8-eb54b7aa5118/2d8cfae4-f7d1-4a7d-b5cb-7588b4c1e8a5"
-					(reference "R14")
+					(reference "R17")
 					(unit 1)
 				)
@@
 		(dnp no)
 		(fields_autoplaced yes)
-		(property "Reference" "R16"
+		(property "Reference" "R19"
 			(at 173.99 116.8399 0)
 			(effects
@@
 			(project "tuner time"
 				(path "/353cef6a-fb6e-40d9-89f8-eb54b7aa5118/2d8cfae4-f7d1-4a7d-b5cb-7588b4c1e8a5"
-					(reference "R16")
-					(unit 1)
-				)
+					(reference "R19")
+					(unit 1)
+				)

Commit message: adding the libraries and the new bom for footprint
Parts:
- C10: MFP CAP_EEE1AA101WR -> EEE1AA101WR
- R18, R19: MFP (none) -> WSTM0805QLR100FNR
Changed lines of the file:
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@@
 			)
 		)
-		(property "MFP" ""
+		(property "MFP" "WSTM0805QLR100FNR"
 			(at 160.02 118.11 0)
 			(effects
@@
 			)
 		)
-		(property "MFP" "CAP_EEE1AA101WR"
+		(property "MFP" "EEE1AA101WR"
 			(at 154.94 64.77 0)
 			(effects
@@
 			)
 		)
-		(property "MFP" ""
+		(property "MFP" "WSTM0805QLR100FNR"
 			(at 171.45 118.11 0)
 			(effects

Commit message: adding the crystal
Parts:
- C10: symbol Device:C_Polarized_US -> GT_LIbrary:C_Polarized_US
- C11, C12, C13, C14, C8, C9: symbol Device:C_Small -> GT_LIbrary:C_Small
- R13, R14, R15, R16, R17, R18, R19, R20: symbol Device:R_US -> GT_LIbrary:R_US
- RV1: symbol Device:R_Potentiometer_US -> GT_LIbrary:R_Potentiometer_US
- U5: symbol DRV8834PWP:DRV8834PWP -> GT_LIbrary:DRV8834PWP
Changed lines of the file:
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@@
 	)
 	(symbol
-		(lib_id "power:GND")
+		(lib_id "GT_LIbrary:GND")
 		(at 256.54 90.17 0)
 		(unit 1)
@@
 	)
 	(symbol
-		(lib_id "Device:R_US")
+		(lib_id "GT_LIbrary:R_US")
 		(at 78.74 58.42 0)
 		(unit 1)
@@
 	)
 	(symbol
-		(lib_id "power:VCC")
+		(lib_id "GT_LIbrary:VCC")
 		(at 245.11 90.17 0)
 		(unit 1)
@@
 	)
 	(symbol
-		(lib_id "Device:R_US")
+		(lib_id "GT_LIbrary:R_US")
 		(at 140.97 120.65 0)
 		(unit 1)
@@
 	)
 	(symbol
-		(lib_id "Device:R_US")
+		(lib_id "GT_LIbrary:R_US")
 		(at 194.31 59.69 90)
 		(unit 1)
@@
 	)
 	(symbol
-		(lib_id "Device:C_Small")
+		(lib_id "GT_LIbrary:C_Small")
 		(at 128.27 72.39 0)
 		(unit 1)
@@
 	)
 	(symbol
-		(lib_id "power:VCC")
+		(lib_id "GT_LIbrary:VCC")
 		(at 163.83 57.15 0)
 		(unit 1)
@@
 	)
 	(symbol
-		(lib_id "power:VCC")
+		(lib_id "GT_LIbrary:VCC")
 		(at 128.27 60.96 0)
 		(unit 1)
@@
 	)
 	(symbol
-		(lib_id "Device:C_Small")
+		(lib_id "GT_LIbrary:C_Small")
 		(at 201.93 64.77 0)
 		(unit 1)
@@
 	)
 	(symbol
-		(lib_id "power:GND")
+		(lib_id "GT_LIbrary:GND")
 		(at 128.27 127 0)
 		(unit 1)
@@
 	)
 	(symbol
-		(lib_id "power:VCC")
+		(lib_id "GT_LIbrary:VCC")
 		(at 78.74 52.07 0)
 		(unit 1)
@@
 	)
 	(symbol
-		(lib_id "power:GND")
+		(lib_id "GT_LIbrary:GND")
 		(at 85.09 120.65 0)
 		(unit 1)
@@
 	)
 	(symbol
-		(lib_id "Device:R_US")
+		(lib_id "GT_LIbrary:R_US")
 		(at 149.86 120.65 0)
 		(unit 1)
@@
 	)
 	(symbol
-		(lib_id "Device:C_Small")
+		(lib_id "GT_LIbrary:C_Small")
 		(at 173.99 64.77 0)
 		(unit 1)
@@
 	)
 	(symbol
-		(lib_id "DRV8834PWP:DRV8834PWP")
+		(lib_id "GT_LIbrary:DRV8834PWP")
 		(at 105.41 81.28 0)
 		(unit 1)
@@
 	)
 	(symbol
-		(lib_id "power:VCC")
+		(lib_id "GT_LIbrary:VCC")
 		(at 238.76 90.17 0)
 		(unit 1)
@@
 	)
 	(symbol
-		(lib_id "Device:C_Small")
+		(lib_id "GT_LIbrary:C_Small")
 		(at 185.42 64.77 0)
 		(unit 1)
@@
 	)
 	(symbol
-		(lib_id "power:GND")
+		(lib_id "GT_LIbrary:GND")
 		(at 163.83 72.39 0)
 		(unit 1)
@@
 	)
 	(symbol
-		(lib_id "Device:C_Small")
+		(lib_id "GT_LIbrary:C_Small")
 		(at 163.83 64.77 0)
 		(unit 1)
@@
 	)
 	(symbol
-		(lib_id "power:VCC")
+		(lib_id "GT_LIbrary:VCC")
 		(at 128.27 116.84 0)
 		(unit 1)
@@
 	)
 	(symbol
-		(lib_id "Device:R_US")
+		(lib_id "GT_LIbrary:R_US")
 		(at 160.02 118.11 0)
 		(unit 1)
@@
 	)
 	(symbol
-		(lib_id "Device:C_Small")
+		(lib_id "GT_LIbrary:C_Small")
 		(at 128.27 121.92 0)
 		(unit 1)
@@
 	)
 	(symbol
-		(lib_id "Device:R_US")
+		(lib_id "GT_LIbrary:R_US")
 		(at 133.35 96.52 90)
 		(unit 1)
@@
 	)
 	(symbol
-		(lib_id "Device:C_Polarized_US")
+		(lib_id "GT_LIbrary:C_Polarized_US")
 		(at 154.94 64.77 0)
 		(unit 1)
@@
 	)
 	(symbol
-		(lib_id "Device:R_US")
+		(lib_id "GT_LIbrary:R_US")
 		(at 152.4 96.52 90)
 		(unit 1)
@@
 	)
 	(symbol
-		(lib_id "Device:R_Potentiometer_US")
+		(lib_id "GT_LIbrary:R_Potentiometer_US")
 		(at 66.04 111.76 0)
 		(mirror x)
@@
 	)
 	(symbol
-		(lib_id "Device:R_US")
+		(lib_id "GT_LIbrary:R_US")
 		(at 171.45 118.11 0)
 		(unit 1)

Commit message: before oscilator
Parts:
- J7: footprint Parts_Library:JST_B4B-XH-A -> B4B-XH-A:JST_B4B-XH-A
- U5: Description_1 (none) -> 11-V, 1.5-A, dual H-bridge or stepper motor driver with 1/3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
Connections:
- net A1: now also U5.4 (AOUT1); no longer U5.1 (AOUT1)
- net A2: now also U5.6 (AOUT2); no longer U5.3 (AOUT2)
- net B1: now also U5.9 (BOUT1); no longer U5.6 (BOUT1)
- net B2: now also U5.7 (BOUT2); no longer U5.4 (BOUT2)
- net DIR: now also U5.12 (DIR); no longer U5.9 (DIR)
- net EN: now also U5.10 (ENBL); no longer U5.7 (ENBL)
- net GND: now also U5.21 (GND); no longer U5.18 (GND)
- net M0: now also U5.13 (M0); no longer U5.10 (M0)
- net M1: now also U5.14 (M1); no longer U5.11 (M1)
- net SLP: now also U5.1 (SLEEP); no longer U5.22 (SLEEP)
- net STEP: now also U5.11 (STEP); no longer U5.8 (STEP)
- net VINT: now also U5.20 (VINT); no longer U5.17 (VINT)
- net VMOT: now also U5.18 (VM), U5.19 (VM); no longer U5.15 (VM), U5.16 (VM)
- net VREF: now also U5.22 (AVREF), U5.23 (BVREF); no longer U5.19 (AVREF), U5.20 (BVREF)
- net at R13.2: now also U5.15 (CONFIG); no longer U5.12 (CONFIG)
- net at R15.1: now also U5.2 (BDECAY); no longer U5.23 (BDECAY)
- net at C8.2: now also U5.17 (VCP); no longer U5.14 (VCP)
- net at R16.1: now also U5.3 (ADECAY); no longer U5.24 (ADECAY)
- net at R14.1: now also U5.16 (FAULT); no longer U5.13 (FAULT)
- net at R19.1: now also U5.5 (AISEN); no longer U5.2 (AISEN)
- net at RV1.3: now also U5.24 (VREF0); no longer U5.21 (VREF0)
- net at R18.1: now also U5.8 (BAISEN); no longer U5.5 (BAISEN)
Changed lines of the file:
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@@
+			)
+		)
+		(property "Description_1" "\n                        \n                            11-V, 1.5-A,  dual H-bridge or stepper motor driver with 1/32 microstep indexer\n                        \n"
+			(at 102.87 124.46 0)
+			(effects
+				(font
+					(size 1.27 1.27)
+				)
+				(justify bottom)
+				(hide yes)
 			)
 		)
@@
 			)
 		)
-		(property "Footprint" "Parts_Library:JST_B4B-XH-A"
+		(property "Footprint" "B4B-XH-A:JST_B4B-XH-A"
 			(at 185.42 83.82 0)
 			(effects

Commit message: added the oscilator
Parts:
- J7: footprint B4B-XH-A:JST_B4B-XH-A -> JST_B4B-XH-A
Changed lines of the file:
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@@
 	(label "A2"
 		(at 175.26 86.36 0)
+		(fields_autoplaced yes)
 		(effects
 			(font
@@
 	(label "A1"
 		(at 128.27 88.9 0)
+		(fields_autoplaced yes)
 		(effects
 			(font
@@
 	(label "B2"
 		(at 128.27 81.28 0)
+		(fields_autoplaced yes)
 		(effects
 			(font
@@
 	(label "A1"
 		(at 175.26 88.9 0)
+		(fields_autoplaced yes)
 		(effects
 			(font
@@
 	(label "A2"
 		(at 128.27 91.44 0)
+		(fields_autoplaced yes)
 		(effects
 			(font
@@
 	(label "B1"
 		(at 128.27 83.82 0)
+		(fields_autoplaced yes)
 		(effects
 			(font
@@
 	(label "B2"
 		(at 175.26 83.82 0)
+		(fields_autoplaced yes)
 		(effects
 			(font
@@
 	(label "B1"
 		(at 175.26 81.28 0)
+		(fields_autoplaced yes)
 		(effects
 			(font
@@
 		(shape input)
 		(at 262.89 88.9 0)
+		(fields_autoplaced yes)
 		(effects
 			(font
@@
 		(shape input)
 		(at 87.63 68.58 180)
+		(fields_autoplaced yes)
 		(effects
 			(font
@@
 		(shape input)
 		(at 87.63 83.82 180)
+		(fields_autoplaced yes)
 		(effects
 			(font
@@
 		(shape input)
 		(at 87.63 91.44 180)
+		(fields_autoplaced yes)
 		(effects
 			(font
@@
 		(shape input)
 		(at 74.93 107.95 90)
+		(fields_autoplaced yes)
 		(effects
 			(font
@@
 		(shape input)
 		(at 245.11 95.25 270)
+		(fields_autoplaced yes)
 		(effects
 			(font
@@
 		(shape input)
 		(at 161.29 96.52 0)
+		(fields_autoplaced yes)
 		(effects
 			(font
@@
 		(shape input)
 		(at 87.63 73.66 180)
+		(fields_autoplaced yes)
 		(effects
 			(font
@@
 		(shape input)
 		(at 87.63 86.36 180)
+		(fields_autoplaced yes)
 		(effects
 			(font
@@
 		(shape input)
 		(at 143.51 99.06 0)
+		(fields_autoplaced yes)
 		(effects
 			(font
@@
 		(shape input)
 		(at 87.63 66.04 180)
+		(fields_autoplaced yes)
 		(effects
 			(font
@@
 		(shape input)
 		(at 238.76 95.25 270)
+		(fields_autoplaced yes)
 		(effects
 			(font
@@
 			)
 		)
-		(property "Footprint" "B4B-XH-A:JST_B4B-XH-A"
+		(property "Footprint" "JST_B4B-XH-A"
 			(at 185.42 83.82 0)
 			(effects

Commit message: before major move
Parts:
- added D3: Green, LED_0805_2012Metric_Pad1.15x1.40mm_HandSolder, symbol GT_LIbrary:LED
- added JP2: SolderJumper_2_Open, Jumper:SolderJumper-2_P1.3mm_Open_RoundedPad1.0x1.5mm, symbol Jumper:SolderJumper_2_Open
- added JP5: M1, Jumper:SolderJumper-3_P1.3mm_Open_RoundedPad1.0x1.5mm, symbol GT_LIbrary:SolderJumper_3_Open
- added JP6: M2, Jumper:SolderJumper-3_P1.3mm_Open_RoundedPad1.0x1.5mm, symbol GT_LIbrary:SolderJumper_3_Open
- added JP7: SLP, Jumper:SolderJumper-3_P1.3mm_Bridged12_RoundedPad1.0x1.5mm, symbol GT_LIbrary:SolderJumper_3_Bridged12
- added R24: 47k, Resistor_SMD:R_0805_2012Metric, symbol GT_LIbrary:R_US
- added R3: 680, Resistor_SMD:R_0805_2012Metric, symbol GT_LIbrary:R_US
- added TP13: ~, TestPoint_THTPad_D0.8mm_Drill0.4mm, symbol GT_LIbrary:TestPoint
Connections:
- net FLT: now also D3.2 (A)
- net GND: now also JP5.3 (B), JP6.3 (B), JP7.3 (B), R3.2
- net M0: now also JP5.2 (C)
- net M1: now also JP6.2 (C)
- net VINT: now also JP5.1 (A), JP6.1 (A), JP7.1 (A)
- net VMOT: now also R24.1
- net VREF: now also TP13.1
- net at R13.2, U5.15 (CONFIG): now also JP2.2 (B)
- net SLP renamed SLEEP
- net SLEEP: now also JP7.2 (C), R24.2
- new net: D3.1 (K), R3.1
- new net Vconfig: JP2.1 (A)

Commit message: Placement done
Parts:
- removed D3: Green, LED_0805_2012Metric_Pad1.15x1.40mm_HandSolder, symbol GT_LIbrary:LED
- removed R3: 680, Resistor_SMD:R_0805_2012Metric, symbol GT_LIbrary:R_US
