File: PCB_v1/MCU.kicad_sch (KiCad schematic)
At the start: 32 parts, among them J10 Conn_01x03, J8 Conn_01x02_Pin, J9 Conn_02x05_Odd_Even, SW8 SW_Push, SW9 SW_SPDT, U6 MAX7375AXR805, U7 STM32F405RGTx

Commit message: before DRC
Connections:
- net SWCLK renamed JTAG_SWCLK
- net SWDIO renamed JTAG_SWDIO
Changed lines of the file:
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@@
 	(wire
 		(pts
-			(xy 66.04 135.89) (xy 81.28 135.89)
+			(xy 66.04 135.89) (xy 86.36 135.89)
 		)
 		(stroke
@@
 		)
 	)
-	(global_label "SWCLK"
+	(global_label "JTAG_SWCLK"
 		(shape output)
 		(at 173.99 100.33 0)
@@
 		)
 		(property "Intersheetrefs" "${INTERSHEET_REFS}"
-			(at 183.2042 100.33 0)
+			(at 188.4656 100.33 0)
 			(effects
 				(font
@@
 		)
 	)
-	(global_label "SWDIO"
+	(global_label "JTAG_SWDIO"
 		(shape bidirectional)
 		(at 173.99 97.79 0)
@@
 		)
 		(property "Intersheetrefs" "${INTERSHEET_REFS}"
-			(at 183.9527 97.79 0)
+			(at 189.2141 97.79 0)
+			(effects
+				(font
+					(size 1.27 1.27)
+				)
+				(justify left)
+				(hide yes)
+			)
+		)
+	)
+	(global_label "JTAG_SWDIO"
+		(shape bidirectional)
+		(at 69.85 133.35 0)
+		(fields_autoplaced yes)
+		(effects
+			(font
+				(size 1.27 1.27)
+			)
+			(justify left)
+		)
+		(property "Intersheetrefs" "${INTERSHEET_REFS}"
+			(at 85.0741 133.35 0)
 			(effects
 				(font
@@
 		)
 	)
-	(global_label "SWDIO"
-		(shape bidirectional)
-		(at 69.85 133.35 0)
-		(fields_autoplaced yes)
-		(effects
-			(font
-				(size 1.27 1.27)
-			)
-			(justify left)
-		)
-		(property "Intersheetrefs" "${INTERSHEET_REFS}"
-			(at 79.8127 133.35 0)
-			(effects
-				(font
-					(size 1.27 1.27)
-				)
-				(justify left)
-				(hide yes)
-			)
-		)
-	)
 	(global_label "PB4"
 		(shape input)
@@
 		)
 	)
-	(global_label "SWCLK"
+	(global_label "JTAG_SWCLK"
 		(shape input)
 		(at 69.85 138.43 0)
@@
 		)
 		(property "Intersheetrefs" "${INTERSHEET_REFS}"
-			(at 79.0642 138.43 0)
+			(at 84.3256 138.43 0)
 			(effects
 				(font
@@
 	(symbol
 		(lib_id "GT_LIbrary:GND")
-		(at 81.28 135.89 0)
+		(at 86.36 135.89 0)
 		(unit 1)
 		(exclude_from_sim no)
@@
 		(fields_autoplaced yes)
 		(property "Reference" "#PWR0107"
-			(at 81.28 142.24 0)
+			(at 86.36 142.24 0)
 			(effects
 				(font
@@
 		)
 		(property "Value" "GND"
-			(at 81.28 140.97 0)
+			(at 86.36 140.97 0)
 			(effects
 				(font
@@
 		)
 		(property "Footprint" ""
-			(at 81.28 135.89 0)
+			(at 86.36 135.89 0)
 			(effects
 				(font
@@
 		)
 		(property "Datasheet" ""
-			(at 81.28 135.89 0)
+			(at 86.36 135.89 0)
 			(effects
 				(font
@@
 		)
 		(property "Description" "Power symbol creates a global label with name \"GND\" , ground"
-			(at 81.28 135.89 0)
+			(at 86.36 135.89 0)
 			(effects
 				(font
