File: PCB_v1/MCU.kicad_sch (KiCad schematic)
At the start: 32 parts, among them J10 Conn_01x03, J8 Conn_01x02_Pin, J9 Conn_02x05_Odd_Even, SW8 SW_Push, SW9 SW_SPDT, U6 MAX7375AXR805, U7 STM32F405RGTx

Commit message: done no text before stiching via
Parts:
- C15, C16, C17, C18, C19, C20, C21, C22, C23, C24: footprint Capacitor_SMD:C_0805_2012Metric -> Library:C_0805_2012Metric
- R21, R22, R23: footprint Resistor_SMD:R_0805_2012Metric -> Library:R_0805_2012Metric
Changed lines of the file:
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@@
 			)
 		)
-		(property "Footprint" "Capacitor_SMD:C_0805_2012Metric"
+		(property "Footprint" "Library:C_0805_2012Metric"
 			(at 42.8752 39.37 0)
 			(effects
@@
 			)
 		)
-		(property "Footprint" "Capacitor_SMD:C_0805_2012Metric"
+		(property "Footprint" "Library:C_0805_2012Metric"
 			(at 117.8052 52.07 0)
 			(effects
@@
 			)
 		)
-		(property "Footprint" "Capacitor_SMD:C_0805_2012Metric"
+		(property "Footprint" "Library:C_0805_2012Metric"
 			(at 129.2352 52.07 0)
 			(effects
@@
 			)
 		)
-		(property "Footprint" "Capacitor_SMD:C_0805_2012Metric"
+		(property "Footprint" "Library:C_0805_2012Metric"
 			(at 122.2248 140.97 0)
 			(effects
@@
 			)
 		)
-		(property "Footprint" "Capacitor_SMD:C_0805_2012Metric"
+		(property "Footprint" "Library:C_0805_2012Metric"
 			(at 94.9452 52.07 0)
 			(effects
@@
 			)
 		)
-		(property "Footprint" "Capacitor_SMD:C_0805_2012Metric"
+		(property "Footprint" "Library:C_0805_2012Metric"
 			(at 106.3752 52.07 0)
 			(effects
@@
 			)
 		)
-		(property "Footprint" "Capacitor_SMD:C_0805_2012Metric"
+		(property "Footprint" "Library:C_0805_2012Metric"
 			(at 140.6652 52.07 0)
 			(effects
@@
 			)
 		)
-		(property "Footprint" "Capacitor_SMD:C_0805_2012Metric"
+		(property "Footprint" "Library:C_0805_2012Metric"
 			(at 84.7852 52.07 0)
 			(effects
@@
 			)
 		)
-		(property "Footprint" "Resistor_SMD:R_0805_2012Metric"
+		(property "Footprint" "Library:R_0805_2012Metric"
 			(at 184.404 112.014 90)
 			(effects
@@
 			)
 		)
-		(property "Footprint" "Resistor_SMD:R_0805_2012Metric"
+		(property "Footprint" "Library:R_0805_2012Metric"
 			(at 88.646 68.834 90)
 			(effects
@@
 			)
 		)
-		(property "Footprint" "Resistor_SMD:R_0805_2012Metric"
+		(property "Footprint" "Library:R_0805_2012Metric"
 			(at 44.704 28.194 90)
 			(effects
@@
 			)
 		)
-		(property "Footprint" "Capacitor_SMD:C_0805_2012Metric"
+		(property "Footprint" "Library:C_0805_2012Metric"
 			(at 63.1952 267.97 0)
 			(effects
@@
 			)
 		)
-		(property "Footprint" "Capacitor_SMD:C_0805_2012Metric"
+		(property "Footprint" "Library:C_0805_2012Metric"
 			(at 132.3848 140.97 0)
 			(effects

Commit message: PCB all Done no Dr.Walter Review
Parts:
- removed R21: 10k, Library:R_0805_2012Metric, symbol GT_LIbrary:R_US
- removed TP7: ~, TestPoint_THTPad_D0.8mm_Drill0.4mm, symbol GT_LIbrary:TestPoint
- added R20: 10k, Library:R_0805_2012Metric, symbol GT_LIbrary:R_US
Connections:
- net BOOT0: now also SW9.2 (B), R20.1
- net GND: now also R20.2; no longer SW9.1 (A)
